File: EMS/Transmitter/substrate/Transmitter.sch (KiCad schematic (older format))
At the start: 8 parts, among them J1 Pico_Left, J2 Pico_Right, J3 ADP_Left, J4 ADP_Right, J5 POWER, J6 EMS_IN, J7 I2C, SW1 SW_SPDT

Commit message: :construction: WIP
Parts:
- J1, J2: symbol Connector:Conn_01x20_Female -> Transmitter-rescue:Conn_01x20_Female-Connector
- J3, J4: symbol Connector:Conn_01x10_Female -> Transmitter-rescue:Conn_01x10_Female-Connector
- J5, J6: symbol Connector:Conn_01x02_Male -> Transmitter-rescue:Conn_01x02_Male-Connector
- J7: symbol Connector:Conn_01x04_Male -> Transmitter-rescue:Conn_01x04_Male-Connector
- SW1: symbol Switch:SW_SPDT -> Transmitter-rescue:SW_SPDT-Switch
Connections:
- net at J1.1 (Pin_1): now also J4.3 (Pin_3)
- net at J1.2 (Pin_2): now also J3.4 (Pin_4)
- net at J2.1 (Pin_1): no longer J4.3 (Pin_3)
- net at J2.2 (Pin_2): no longer J3.4 (Pin_4)
Other:
- note removed: "RX"
- note removed: "TX"
Changed lines of the file:
@@
 $EndDescr
 $Comp
-L Connector:Conn_01x20_Female J1
+L Transmitter-rescue:Conn_01x20_Female-Connector J1
 U 1 1 60B0492F
 P 4350 3700
@@
 $EndComp
 $Comp
-L Connector:Conn_01x20_Female J2
+L Transmitter-rescue:Conn_01x20_Female-Connector J2
 U 1 1 60B063B8
 P 4650 3800
@@
 $EndComp
 $Comp
-L Connector:Conn_01x10_Female J3
+L Transmitter-rescue:Conn_01x10_Female-Connector J3
 U 1 1 60B0F59A
 P 6450 3200
@@
 $EndComp
 $Comp
-L Connector:Conn_01x10_Female J4
+L Transmitter-rescue:Conn_01x10_Female-Connector J4
 U 1 1 60B10C64
 P 6700 3200
@@
 $EndComp
 $Comp
-L power:+5V #PWR0101
+L Transmitter-rescue:+5V-power #PWR0101
 U 1 1 60B12616
 P 5950 2350
@@
 NoConn ~ 4850 2800
 $Comp
-L power:GND #PWR0102
+L Transmitter-rescue:GND-power #PWR0102
 U 1 1 60B3440B
 P 5950 5000
@@
 NoConn ~ 4150 3100
 NoConn ~ 4150 3000
-NoConn ~ 4150 2900
-NoConn ~ 4150 2800
 NoConn ~ 4850 3000
 NoConn ~ 4850 3100
@@
 	6950 3600 6900 3600
 $Comp
-L Connector:Conn_01x02_Male J5
+L Transmitter-rescue:Conn_01x02_Male-Connector J5
 U 1 1 60C2BF9E
 P 2800 4450
@@
 $EndComp
 $Comp
-L power:+5V #PWR01
+L Transmitter-rescue:+5V-power #PWR01
 U 1 1 60C2C475
 P 3350 4300
@@
 $EndComp
 $Comp
-L power:GND #PWR02
+L Transmitter-rescue:GND-power #PWR02
 U 1 1 60C2CC2C
 P 3350 4700
@@
 	5150 3600 6250 3600
 $Comp
-L Connector:Conn_01x02_Male J6
+L Transmitter-rescue:Conn_01x02_Male-Connector J6
 U 1 1 60B16252
 P 7400 4100
@@
 NoConn ~ 4150 4300
 NoConn ~ 4150 4400
-Text Notes 4800 4700 0    50   ~ 0
-TX
-Text Notes 4800 4600 0    50   ~ 0
-RX
 Wire Wire Line
 	5150 3200 5150 3600
-Wire Wire Line
-	4850 4700 7050 4700
-Wire Wire Line
-	6150 3100 6150 4600
-Wire Wire Line
-	4850 4600 6150 4600
 Wire Wire Line
 	4850 4400 6050 4400
@@
 Wire Wire Line
 	4850 4200 7200 4200
-Wire Wire Line
-	7050 4700 7050 3000
-$Comp
-L Switch:SW_SPDT SW1
+$Comp
+L Transmitter-rescue:SW_SPDT-Switch SW1
 U 1 1 60B2577F
 P 5450 2900
@@
 NoConn ~ 5650 2800
 $Comp
-L Connector:Conn_01x04_Male J7
+L Transmitter-rescue:Conn_01x04_Male-Connector J7
 U 1 1 60B4044F
 P 3550 3300
@@
 Wire Wire Line
 	3900 4850 4950 4850
+Wire Wire Line
+	7050 3000 7050 2450
+Wire Wire Line
+	7050 2450 4100 2450
+Wire Wire Line
+	4100 2450 4100 2800
+Wire Wire Line
+	4100 2800 4150 2800
+Wire Wire Line
+	4150 2900 4050 2900
+Wire Wire Line
+	4050 2900 4050 2500
+Wire Wire Line
+	4050 2500 6150 2500
+Wire Wire Line
+	6150 2500 6150 3100
+NoConn ~ 4850 4600
+NoConn ~ 4850 4700
 $EndSCHEMATC

Commit message: 基板の更新
Parts:
- J1, J2: symbol Transmitter-rescue:Conn_01x20_Female-Connector -> Transmitter-rescue:Conn_01x20_Female-Connector-Transmitter-rescue
- J3, J4: symbol Transmitter-rescue:Conn_01x10_Female-Connector -> Transmitter-rescue:Conn_01x10_Female-Connector-Transmitter-rescue
- J5, J6: symbol Transmitter-rescue:Conn_01x02_Male-Connector -> Transmitter-rescue:Conn_01x02_Male-Connector-Transmitter-rescue
- J7: symbol Transmitter-rescue:Conn_01x04_Male-Connector -> Transmitter-rescue:Conn_01x04_Male-Connector-Transmitter-rescue
- SW1: symbol Transmitter-rescue:SW_SPDT-Switch -> Transmitter-rescue:SW_SPDT-Switch-Transmitter-rescue
Changed lines of the file:
@@
 $EndDescr
 $Comp
-L Transmitter-rescue:Conn_01x20_Female-Connector J1
+L Transmitter-rescue:Conn_01x20_Female-Connector-Transmitter-rescue J1
 U 1 1 60B0492F
 P 4350 3700
@@
 $EndComp
 $Comp
-L Transmitter-rescue:Conn_01x20_Female-Connector J2
+L Transmitter-rescue:Conn_01x20_Female-Connector-Transmitter-rescue J2
 U 1 1 60B063B8
 P 4650 3800
@@
 $EndComp
 $Comp
-L Transmitter-rescue:Conn_01x10_Female-Connector J3
+L Transmitter-rescue:Conn_01x10_Female-Connector-Transmitter-rescue J3
 U 1 1 60B0F59A
 P 6450 3200
@@
 $EndComp
 $Comp
-L Transmitter-rescue:Conn_01x10_Female-Connector J4
+L Transmitter-rescue:Conn_01x10_Female-Connector-Transmitter-rescue J4
 U 1 1 60B10C64
 P 6700 3200
@@
 $EndComp
 $Comp
-L Transmitter-rescue:+5V-power #PWR0101
+L Transmitter-rescue:+5V-power-Transmitter-rescue #PWR0101
 U 1 1 60B12616
 P 5950 2350
@@
 NoConn ~ 4850 2800
 $Comp
-L Transmitter-rescue:GND-power #PWR0102
+L Transmitter-rescue:GND-power-Transmitter-rescue #PWR0102
 U 1 1 60B3440B
 P 5950 5000
@@
 	6950 3600 6900 3600
 $Comp
-L Transmitter-rescue:Conn_01x02_Male-Connector J5
+L Transmitter-rescue:Conn_01x02_Male-Connector-Transmitter-rescue J5
 U 1 1 60C2BF9E
 P 2800 4450
@@
 $EndComp
 $Comp
-L Transmitter-rescue:+5V-power #PWR01
+L Transmitter-rescue:+5V-power-Transmitter-rescue #PWR01
 U 1 1 60C2C475
 P 3350 4300
@@
 $EndComp
 $Comp
-L Transmitter-rescue:GND-power #PWR02
+L Transmitter-rescue:GND-power-Transmitter-rescue #PWR02
 U 1 1 60C2CC2C
 P 3350 4700
@@
 	5150 3600 6250 3600
 $Comp
-L Transmitter-rescue:Conn_01x02_Male-Connector J6
+L Transmitter-rescue:Conn_01x02_Male-Connector-Transmitter-rescue J6
 U 1 1 60B16252
 P 7400 4100
@@
 	4850 4200 7200 4200
 $Comp
-L Transmitter-rescue:SW_SPDT-Switch SW1
+L Transmitter-rescue:SW_SPDT-Switch-Transmitter-rescue SW1
 U 1 1 60B2577F
 P 5450 2900
@@
 NoConn ~ 5650 2800
 $Comp
-L Transmitter-rescue:Conn_01x04_Male-Connector J7
+L Transmitter-rescue:Conn_01x04_Male-Connector-Transmitter-rescue J7
 U 1 1 60B4044F
 P 3550 3300

Commit message: Update transmitter.
Parts:
- removed J1: Pico_Left, Connector_PinSocket_2.54mm:PinSocket_1x20_P2.54mm_Vertical, symbol Transmitter-rescue:Conn_01x20_Female-Connector-Transmitter-rescue
- removed J2: Pico_Right, Connector_PinSocket_2.54mm:PinSocket_1x20_P2.54mm_Vertical, symbol Transmitter-rescue:Conn_01x20_Female-Connector-Transmitter-rescue
- removed J7: I2C, Connector_JST:JST_XH_S4B-XH-A_1x04_P2.50mm_Horizontal, symbol Transmitter-rescue:Conn_01x04_Male-Connector-Transmitter-rescue
- added R1, R2, R3: 18Ω, Resistor_THT:R_Axial_DIN0207_L6.3mm_D2.5mm_P7.62mm_Horizontal, symbol Device:R
- added U1: SeeeduinoXIAO, Seeeduino XIAO KICAD:Seeeduino XIAO-MOUDLE14P-2.54-21X17.8MM, symbol Seeeduino_XIAO:SeeeduinoXIAO
- J3: value ADP_Left -> ADP_L; symbol Transmitter-rescue:Conn_01x10_Female-Connector-Transmitter-rescue -> Transmitter-rescue:Conn_01x10_Female-Connector-Transmitter-rescue-Transmitter-rescue
- J4: value ADP_Right -> ADP_R; symbol Transmitter-rescue:Conn_01x10_Female-Connector-Transmitter-rescue -> Transmitter-rescue:Conn_01x10_Female-Connector-Transmitter-rescue-Transmitter-rescue
- J5: symbol Transmitter-rescue:Conn_01x02_Male-Connector-Transmitter-rescue -> Transmitter-rescue:Conn_01x02_Male-Connector-Transmitter-rescue-Transmitter-rescue
- J6: value EMS_IN -> ESS_IN; symbol Transmitter-rescue:Conn_01x02_Male-Connector-Transmitter-rescue -> Transmitter-rescue:Conn_01x02_Male-Connector-Transmitter-rescue-Transmitter-rescue
- SW1: symbol Transmitter-rescue:SW_SPDT-Switch-Transmitter-rescue -> Transmitter-rescue:SW_SPDT-Switch-Transmitter-rescue-Transmitter-rescue
Connections:
- net +5V: now also J6.1 (Pin_1), SW1.1 (A), R3.1, U1.14 (5V); no longer J5.1 (Pin_1), SW1.3 (C)
- net GND: now also R1.2, U1.13 (GND)
- net TX: now reaches J4.3 (Pin_3)
- net TX: now also U1.7 (PB08_A6_D6_TX)
- net RX: now reaches J3.4 (Pin_4)
- net RX: now also U1.8 (PB09_A7_D7_RX)
- net +3V3: now reaches J3.9 (Pin_9)
- net +3V3: now also U1.12 (3V3)
- net PW_IN: now reaches SW1.2 (B)
- net PW_IN: now also J5.1 (Pin_1)
- net ESS_IN: now reaches J6.2 (Pin_2)
- net ESS_IN: now also U1.2 (PA4_A1_D1)
- new net: R1.1, R2.2
- new net: R2.1, R3.2
- no-connect marks 43 -> 31
Other:
- note added: "Dummy_load"
- note added: "ESS"
- note added: "IM920-ADP"
- note added: "Power"
- note added: "Power_SW"
- note added: "RST"
- note added: "RTS"
- note added: "RxD"
- note added: "SeeeduinoXIAO"
- note added: "TxD"
- moved on the sheet: J3, J4, J5, J6, SW1
