File: EMS/Receiver/substrate/Receiver.sch (KiCad schematic (older format))
At the start: 14 parts, among them J1 F303k8_Left, J10 3V3_OUT, J2 F303k8_Right, J3 ADP_Left, J4 ADP_Right, J5 Power_IN, J6 EMS_OUT, J7 CAN, J8 I2C, J9 UART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

Commit message: :construction: WIP
Parts:
- removed J9: UART, Connector_JST:JST_XH_S2B-XH-A_1x02_P2.50mm_Horizontal, symbol Connector:Conn_01x02_Male
- D1, D2: symbol Device:LED -> Receiver-rescue:LED-Device
- J1, J2: symbol Connector:Conn_01x15_Female -> Receiver-rescue:Conn_01x15_Female-Connector
- J10, J5, J6, J7, J8: symbol Connector:Conn_01x02_Male -> Receiver-rescue:Conn_01x02_Male-Connector
- J3, J4: symbol Connector:Conn_01x10_Female -> Receiver-rescue:Conn_01x10_Female-Connector
- SW1: symbol Switch:SW_SPDT -> Receiver-rescue:SW_SPDT-Switch
- U1: symbol Isolator:LTV-817 -> Receiver-rescue:LTV-817-Isolator
Connections:
- net at J1.1 (Pin_1): now also J4.3 (Pin_3)
- net at J1.2 (Pin_2): now also J3.4 (Pin_4)
- net at J2.10 (Pin_10): no longer J3.4 (Pin_4)
- net at J2.12 (Pin_12): no longer J3.1 (Pin_1)
- net at J2.15 (Pin_15): now also J3.1 (Pin_1); no longer J4.3 (Pin_3)
- no-connect marks 31 -> 33
Changed lines of the file:
@@
 $EndDescr
 $Comp
-L Connector:Conn_01x15_Female J2
-U 1 1 60AEFA8A
-P 4750 3050
-F 0 "J2" H 4600 2250 50  0000 C CNN
-F 1 "F303k8_Right" H 4550 3900 50  0000 C CNN
-F 2 "Connector_PinSocket_2.54mm:PinSocket_1x15_P2.54mm_Vertical" H 4750 3050 50  0001 C CNN
-F 3 "~" H 4750 3050 50  0001 C CNN
-	1    4750 3050
-	-1   0    0    -1
-$EndComp
-$Comp
-L power:GND #PWR0101
+L Receiver-rescue:GND-power #PWR0101
 U 1 1 60AF1801
 P 2800 4900
@@
 $EndComp
 $Comp
-L Connector:Conn_01x15_Female J1
-U 1 1 60AEE444
-P 4550 3050
-F 0 "J1" H 4350 2250 50  0000 L CNN
-F 1 "F303k8_Left" H 4200 3900 50  0000 L CNN
-F 2 "Connector_PinSocket_2.54mm:PinSocket_1x15_P2.54mm_Vertical" H 4550 3050 50  0001 C CNN
-F 3 "~" H 4550 3050 50  0001 C CNN
-	1    4550 3050
-	1    0    0    -1
-$EndComp
-$Comp
-L Connector:Conn_01x10_Female J3
+L Receiver-rescue:Conn_01x10_Female-Connector J3
 U 1 1 60B01E56
 P 7550 2850
@@
 $EndComp
 $Comp
-L Connector:Conn_01x10_Female J4
+L Receiver-rescue:Conn_01x10_Female-Connector J4
 U 1 1 60B038BF
 P 7750 2850
@@
 	7950 3250 8150 3250
 $Comp
-L Connector:Conn_01x02_Male J5
+L Receiver-rescue:Conn_01x02_Male-Connector J5
 U 1 1 60B39C1D
 P 2100 4650
@@
 RX
 $Comp
-L Connector:Conn_01x02_Male J7
+L Receiver-rescue:Conn_01x02_Male-Connector J7
 U 1 1 60B5D24A
 P 3000 3450
@@
 CAN_TD
 $Comp
-L Isolator:LTV-817 U1
+L Receiver-rescue:LTV-817-Isolator U1
 U 1 1 60AF1260
 P 6400 3200
@@
 	0    -1   1    0
 $EndComp
-Wire Wire Line
-	8150 2250 8150 2650
-$Comp
-L Device:LED D1
+$Comp
+L Receiver-rescue:LED-Device D1
 U 1 1 60B360E0
 P 6700 3850
@@
 $EndComp
 $Comp
-L Switch:SW_SPDT SW1
+L Receiver-rescue:SW_SPDT-Switch SW1
 U 1 1 60B49C25
 P 7250 3950
@@
 	6850 3850 7050 3850
 $Comp
-L Device:LED D2
+L Receiver-rescue:LED-Device D2
 U 1 1 60B97B28
 P 6700 4050
@@
 	6550 4050 6300 4050
 $Comp
-L Connector:Conn_01x02_Male J6
+L Receiver-rescue:Conn_01x02_Male-Connector J6
 U 1 1 60BC7FBD
 P 8500 3950
@@
 Wire Wire Line
 	8300 3950 7450 3950
-$Comp
-L Connector:Conn_01x02_Male J9
-U 1 1 60CFA959
-P 3000 2350
-F 0 "J9" H 3100 2550 50  0000 C CNN
-F 1 "UART" H 3100 2450 50  0000 C CNN
-F 2 "Connector_JST:JST_XH_S2B-XH-A_1x02_P2.50mm_Horizontal" H 3000 2350 50  0001 C CNN
-F 3 "~" H 3000 2350 50  0001 C CNN
-	1    3000 2350
-	1    0    0    -1
-$EndComp
-Wire Wire Line
-	3200 2350 4350 2350
-Wire Wire Line
-	4350 2450 3200 2450
 NoConn ~ 4950 2750
 NoConn ~ 4350 2850
@@
 	5950 4850 5950 5000
 $Comp
-L power:GND #PWR0102
+L Receiver-rescue:GND-power #PWR0102
 U 1 1 60AFF5CE
 P 5950 5000
@@
 	7500 4050 8300 4050
 $Comp
-L Connector:Conn_01x02_Male J8
+L Receiver-rescue:Conn_01x02_Male-Connector J8
 U 1 1 60CEE284
 P 3000 2950
@@
 	3200 3450 4000 3450
 $Comp
-L power:+5V #PWR0103
+L Receiver-rescue:+5V-power #PWR0103
 U 1 1 60B37161
 P 5750 1550
@@
 $EndComp
 $Comp
-L power:+5V #PWR0104
+L Receiver-rescue:+5V-power #PWR0104
 U 1 1 60B5796E
 P 2800 4500
@@
 	3200 3050 4350 3050
 $Comp
-L Connector:Conn_01x02_Male J10
+L Receiver-rescue:Conn_01x02_Male-Connector J10
 U 1 1 60B21E10
 P 8500 4450
@@
 	7500 4050 7500 4200
 Wire Wire Line
-	4950 3750 5200 3750
-Wire Wire Line
-	4950 3250 5300 3250
-Wire Wire Line
 	5100 2450 5100 4850
 Connection ~ 5100 4850
@@
 	5100 4850 5950 4850
 Wire Wire Line
-	5300 3250 5300 2750
-Wire Wire Line
-	5300 2750 7350 2750
-Wire Wire Line
-	4950 3450 5400 3450
-Wire Wire Line
-	5200 2250 5200 3750
-Wire Wire Line
-	5200 2250 8150 2250
-Wire Wire Line
-	5400 2450 5400 3450
-Wire Wire Line
-	5400 2450 7350 2450
-Wire Wire Line
 	4950 2650 5750 2650
 Wire Wire Line
 	5750 1550 5750 2650
+Wire Wire Line
+	4150 2350 4150 2050
+Wire Wire Line
+	4150 2050 8150 2050
+Wire Wire Line
+	4150 2350 4350 2350
+Wire Wire Line
+	8150 2050 8150 2650
+Wire Wire Line
+	4350 2450 3850 2450
+Wire Wire Line
+	3850 2450 3850 1900
+Wire Wire Line
+	3850 1900 6800 1900
+Wire Wire Line
+	6800 1900 6800 2750
+Wire Wire Line
+	6800 2750 7350 2750
+NoConn ~ 4950 3450
+NoConn ~ 4950 3250
+Wire Wire Line
+	7350 2450 5250 2450
+Wire Wire Line
+	5250 2450 5250 3750
+Wire Wire Line
+	5250 3750 4950 3750
+$Comp
+L Receiver-rescue:Conn_01x15_Female-Connector J2
+U 1 1 60AEFA8A
+P 4750 3050
+F 0 "J2" H 4600 2250 50  0000 C CNN
+F 1 "F303k8_Right" H 4550 3900 50  0000 C CNN
+F 2 "Connector_PinSocket_2.54mm:PinSocket_1x15_P2.54mm_Vertical" H 4750 3050 50  0001 C CNN
+F 3 "~" H 4750 3050 50  0001 C CNN
+	1    4750 3050
+	-1   0    0    -1
+$EndComp
+$Comp
+L Receiver-rescue:Conn_01x15_Female-Connector J1
+U 1 1 60AEE444
+P 4550 3050
+F 0 "J1" H 4350 2250 50  0000 L CNN
+F 1 "F303k8_Left" H 4200 3900 50  0000 L CNN
+F 2 "Connector_PinSocket_2.54mm:PinSocket_1x15_P2.54mm_Vertical" H 4550 3050 50  0001 C CNN
+F 3 "~" H 4550 3050 50  0001 C CNN
+	1    4550 3050
+	1    0    0    -1
+$EndComp
 $EndSCHEMATC

Commit message: 基板の更新
Parts:
- D1, D2: symbol Receiver-rescue:LED-Device -> Receiver-rescue:LED-Device-Receiver-rescue
- J1, J2: symbol Receiver-rescue:Conn_01x15_Female-Connector -> Receiver-rescue:Conn_01x15_Female-Connector-Receiver-rescue
- J10, J5, J6, J7, J8: symbol Receiver-rescue:Conn_01x02_Male-Connector -> Receiver-rescue:Conn_01x02_Male-Connector-Receiver-rescue
- J3, J4: symbol Receiver-rescue:Conn_01x10_Female-Connector -> Receiver-rescue:Conn_01x10_Female-Connector-Receiver-rescue
- SW1: footprint Button_Switch_THT:SW_Slide_1P2T_CK_OS102011MS2Q -> Connector_PinHeader_2.54mm:PinHeader_1x03_P2.54mm_Vertical; symbol Receiver-rescue:SW_SPDT-Switch -> Receiver-rescue:SW_SPDT-Switch-Receiver-rescue
- U1: symbol Receiver-rescue:LTV-817-Isolator -> Receiver-rescue:LTV-817-Isolator-Receiver-rescue
Changed lines of the file:
@@
 $EndDescr
 $Comp
-L Receiver-rescue:GND-power #PWR0101
+L Receiver-rescue:GND-power-Receiver-rescue #PWR0101
 U 1 1 60AF1801
 P 2800 4900
@@
 $EndComp
 $Comp
-L Receiver-rescue:Conn_01x10_Female-Connector J3
+L Receiver-rescue:Conn_01x10_Female-Connector-Receiver-rescue J3
 U 1 1 60B01E56
 P 7550 2850
@@
 $EndComp
 $Comp
-L Receiver-rescue:Conn_01x10_Female-Connector J4
+L Receiver-rescue:Conn_01x10_Female-Connector-Receiver-rescue J4
 U 1 1 60B038BF
 P 7750 2850
@@
 	7950 3250 8150 3250
 $Comp
-L Receiver-rescue:Conn_01x02_Male-Connector J5
+L Receiver-rescue:Conn_01x02_Male-Connector-Receiver-rescue J5
 U 1 1 60B39C1D
 P 2100 4650
@@
 RX
 $Comp
-L Receiver-rescue:Conn_01x02_Male-Connector J7
+L Receiver-rescue:Conn_01x02_Male-Connector-Receiver-rescue J7
 U 1 1 60B5D24A
 P 3000 3450
@@
 CAN_TD
 $Comp
-L Receiver-rescue:LTV-817-Isolator U1
+L Receiver-rescue:LTV-817-Isolator-Receiver-rescue U1
 U 1 1 60AF1260
 P 6400 3200
@@
 $EndComp
 $Comp
-L Receiver-rescue:LED-Device D1
+L Receiver-rescue:LED-Device-Receiver-rescue D1
 U 1 1 60B360E0
 P 6700 3850
@@
 $EndComp
 $Comp
-L Receiver-rescue:SW_SPDT-Switch SW1
+L Receiver-rescue:SW_SPDT-Switch-Receiver-rescue SW1
 U 1 1 60B49C25
 P 7250 3950
 F 0 "SW1" H 7250 4235 50  0000 C CNN
 F 1 "SW_SPDT" H 7250 4144 50  0000 C CNN
-F 2 "Button_Switch_THT:SW_Slide_1P2T_CK_OS102011MS2Q" H 7250 3950 50  0001 C CNN
+F 2 "Connector_PinHeader_2.54mm:PinHeader_1x03_P2.54mm_Vertical" H 7250 3950 50  0001 C CNN
 F 3 "~" H 7250 3950 50  0001 C CNN
 	1    7250 3950
@@
 	6850 3850 7050 3850
 $Comp
-L Receiver-rescue:LED-Device D2
+L Receiver-rescue:LED-Device-Receiver-rescue D2
 U 1 1 60B97B28
 P 6700 4050
@@
 	6550 4050 6300 4050
 $Comp
-L Receiver-rescue:Conn_01x02_Male-Connector J6
+L Receiver-rescue:Conn_01x02_Male-Connector-Receiver-rescue J6
 U 1 1 60BC7FBD
 P 8500 3950
@@
 	5950 4850 5950 5000
 $Comp
-L Receiver-rescue:GND-power #PWR0102
+L Receiver-rescue:GND-power-Receiver-rescue #PWR0102
 U 1 1 60AFF5CE
 P 5950 5000
@@
 	7500 4050 8300 4050
 $Comp
-L Receiver-rescue:Conn_01x02_Male-Connector J8
+L Receiver-rescue:Conn_01x02_Male-Connector-Receiver-rescue J8
 U 1 1 60CEE284
 P 3000 2950
@@
 	3200 3450 4000 3450
 $Comp
-L Receiver-rescue:+5V-power #PWR0103
+L Receiver-rescue:+5V-power-Receiver-rescue #PWR0103
 U 1 1 60B37161
 P 5750 1550
@@
 $EndComp
 $Comp
-L Receiver-rescue:+5V-power #PWR0104
+L Receiver-rescue:+5V-power-Receiver-rescue #PWR0104
 U 1 1 60B5796E
 P 2800 4500
@@
 	3200 3050 4350 3050
 $Comp
-L Receiver-rescue:Conn_01x02_Male-Connector J10
+L Receiver-rescue:Conn_01x02_Male-Connector-Receiver-rescue J10
 U 1 1 60B21E10
 P 8500 4450
@@
 	5250 3750 4950 3750
 $Comp
-L Receiver-rescue:Conn_01x15_Female-Connector J2
+L Receiver-rescue:Conn_01x15_Female-Connector-Receiver-rescue J2
 U 1 1 60AEFA8A
 P 4750 3050
@@
 $EndComp
 $Comp
-L Receiver-rescue:Conn_01x15_Female-Connector J1
+L Receiver-rescue:Conn_01x15_Female-Connector-Receiver-rescue J1
 U 1 1 60AEE444
 P 4550 3050

Commit message: Update Receiver.
Parts:
- removed J1: F303k8_Left, Connector_PinSocket_2.54mm:PinSocket_1x15_P2.54mm_Vertical, symbol Receiver-rescue:Conn_01x15_Female-Connector-Receiver-rescue
- removed J10: 3V3_OUT, Connector_JST:JST_XH_S2B-XH-A_1x02_P2.50mm_Horizontal, symbol Receiver-rescue:Conn_01x02_Male-Connector-Receiver-rescue
- removed J2: F303k8_Right, Connector_PinSocket_2.54mm:PinSocket_1x15_P2.54mm_Vertical, symbol Receiver-rescue:Conn_01x15_Female-Connector-Receiver-rescue
- removed J7: CAN, Connector_JST:JST_XH_S2B-XH-A_1x02_P2.50mm_Horizontal, symbol Receiver-rescue:Conn_01x02_Male-Connector-Receiver-rescue
- removed J8: I2C, Connector_JST:JST_XH_S2B-XH-A_1x02_P2.50mm_Horizontal, symbol Receiver-rescue:Conn_01x02_Male-Connector-Receiver-rescue
- added D3, D4: LED, LED_THT:LED_D5.0mm, symbol Receiver-rescue:LED-Device-Receiver-rescue-Receiver-rescue
- added J1: RESS_OUT2, Connector_JST:JST_XH_S2B-XH-A_1x02_P2.50mm_Horizontal, symbol Receiver-rescue:Conn_01x02_Male-Connector-Receiver-rescue-Receiver-rescue
- added SW2: SW_SPDT, Connector_PinHeader_2.54mm:PinHeader_1x03_P2.54mm_Vertical, symbol Receiver-rescue:SW_SPDT-Switch-Receiver-rescue-Receiver-rescue
- added U2: SeeeduinoXIAO, Seeeduino XIAO KICAD:Seeeduino XIAO-MOUDLE14P-2.54-21X17.8MM, symbol Seeeduino_XIAO:SeeeduinoXIAO
- added U3: LTV-817, Package_DIP:DIP-4_W7.62mm, symbol Receiver-rescue:LTV-817-Isolator-Receiver-rescue-Receiver-rescue
- D1, D2: symbol Receiver-rescue:LED-Device-Receiver-rescue -> Receiver-rescue:LED-Device-Receiver-rescue-Receiver-rescue
- J3: value ADP_Left -> ADP_L; symbol Receiver-rescue:Conn_01x10_Female-Connector-Receiver-rescue -> Receiver-rescue:Conn_01x10_Female-Connector-Receiver-rescue-Receiver-rescue
- J4: value ADP_Right -> ADP_R; symbol Receiver-rescue:Conn_01x10_Female-Connector-Receiver-rescue -> Receiver-rescue:Conn_01x10_Female-Connector-Receiver-rescue-Receiver-rescue
- J5: symbol Receiver-rescue:Conn_01x02_Male-Connector-Receiver-rescue -> Receiver-rescue:Conn_01x02_Male-Connector-Receiver-rescue-Receiver-rescue
- J6: value EMS_OUT -> RESS_OUT1; symbol Receiver-rescue:Conn_01x02_Male-Connector-Receiver-rescue -> Receiver-rescue:Conn_01x02_Male-Connector-Receiver-rescue-Receiver-rescue
- SW1: symbol Receiver-rescue:SW_SPDT-Switch-Receiver-rescue -> Receiver-rescue:SW_SPDT-Switch-Receiver-rescue-Receiver-rescue
- U1: symbol Receiver-rescue:LTV-817-Isolator-Receiver-rescue -> Receiver-rescue:LTV-817-Isolator-Receiver-rescue-Receiver-rescue
Connections:
- net +5V: now also U2.14 (5V)
- net GND: now also U2.13 (GND), U3.2
- net TX: now reaches J4.3 (Pin_3)
- net TX: now also U2.7 (PB08_A6_D6_TX)
- net RX: now reaches J3.4 (Pin_4)
- net RX: now also U2.8 (PB09_A7_D7_RX)
- net +3V3: now reaches J3.9 (Pin_9)
- net +3V3: now also U2.12 (3V3)
- net Out1: now reaches U1.1
- net Out1: now also U2.3 (PA10_A2_D2)
- new net: D3.2 (A), U3.3
- new net: D4.2 (A), J1.2 (Pin_2), U3.4
- new net: D3.1 (K), SW2.1 (A)
- new net: J1.1 (Pin_1), SW2.2 (B)
- new net: D4.1 (K), SW2.3 (C)
- new net Out2: U2.4 (PA11_A3_D3), U3.1
- no-connect marks 33 -> 29
Other:
- note added: "IM920-ADP"
- note added: "Power"
- note added: "SeeeduinoXIAO"
- note added: "Status_SW1"
- note added: "Status_SW2"
- note removed: "CAN_RD"
- note removed: "CAN_TD"
- note removed: "CTS"
- note removed: "SCL"
- note removed: "SDA"
- note removed: "TX\n"
- moved on the sheet: D1, D2, J3, J4, J5, J6, SW1, U1
