File: EMS/Receiver/substrate/Receiver.kicad_pcb (KiCad board)
At the start: 2 copper layers, 81.3 x 61 mm, 18 parts, among them SW1 SW_SPDT, U1 LTV-817

Commit message: 基板の更新
Parts:
- removed OUT 3.3V: 3V3_OUT, Connector_JST:JST_XH_S2B-XH-A_1x02_P2.50mm_Horizontal
- removed the REF** at (158.8, 148.6)
- removed the REF** at (85.1, 148.6)
- removed the REF** at (158.8, 95.2)
- removed the REF** at (85.1, 95.2)
- removed UART: UART, Connector_JST:JST_XH_S2B-XH-A_1x02_P2.50mm_Horizontal
- added 3.3V OUT: 3V3_OUT, Connector_JST:JST_XH_S2B-XH-A_1x02_P2.50mm_Horizontal, F.Cu at (152.4, 130.8)
- added REF**: MountingHole_3.2mm_M3, MountingHole:MountingHole_3.2mm_M3, F.Cu at (159.0, 149.0)
- added REF**: MountingHole_3.2mm_M3, MountingHole:MountingHole_3.2mm_M3, F.Cu at (159.0, 95.0)
- added REF**: MountingHole_3.2mm_M3, MountingHole:MountingHole_3.2mm_M3, F.Cu at (85.0, 95.0)
- added REF**: MountingHole_3.2mm_M3, MountingHole:MountingHole_3.2mm_M3, F.Cu at (85.0, 149.0)
- SW1: footprint Button_Switch_THT:SW_Slide_1P2T_CK_OS102011MS2Q -> Connector_PinHeader_2.54mm:PinHeader_1x03_P2.54mm_Vertical
- moved CAN 11.4 mm to (152.8, 105.4)
- moved I2C 11.4 mm to (152.4, 118.1)
- moved SW1 0.54 mm to (91.4, 147.3), turned to 90 degrees
- renumbered ON to OFF, OFF to ON
Connections:
- L pad 10: (no net) -> Net-(J1-Pad10)
- L pad 11: (no net) -> Net-(J1-Pad11)
- L pad 12: (no net) -> Net-(J1-Pad12)
- L pad 14: (no net) -> Net-(J1-Pad14)
- L pad 15: (no net) -> Net-(J1-Pad15)
- L pad 3: (no net) -> Net-(J1-Pad3)
- L pad 6: (no net) -> Net-(J1-Pad6)
- L pad 9: (no net) -> Net-(J1-Pad9)
- L pad 1: Net-(J2-Pad12) -> Net-(J2-Pad15)
- L pad 10: (no net) -> Net-(J3-Pad10)
- L pad 2: (no net) -> Net-(J3-Pad2)
- L pad 3: (no net) -> Net-(J3-Pad3)
- L pad 4: Net-(J2-Pad10) -> Net-(J1-Pad2)
- L pad 5: (no net) -> Net-(J3-Pad5)
- L pad 6: (no net) -> Net-(J3-Pad6)
- L pad 7: (no net) -> Net-(J3-Pad7)
- L pad 8: (no net) -> Net-(J3-Pad8)
- R pad 1: (no net) -> Net-(J2-Pad1)
- R pad 11: (no net) -> Net-(J2-Pad11)
- R pad 13: (no net) -> Net-(J2-Pad13)
- R pad 3: (no net) -> Net-(J2-Pad3)
- R pad 5: (no net) -> Net-(J2-Pad5)
- R pad 7: (no net) -> Net-(J2-Pad7)
- R pad 8: (no net) -> Net-(J2-Pad8)
- R pad 9: (no net) -> Net-(J2-Pad9)
- R pad 1: (no net) -> Net-(J4-Pad1)
- R pad 10: (no net) -> Net-(J4-Pad10)
- R pad 2: (no net) -> Net-(J4-Pad2)
- R pad 3: Net-(J2-Pad15) -> Net-(J1-Pad1)
- R pad 4: (no net) -> Net-(J4-Pad4)
- R pad 5: (no net) -> Net-(J4-Pad5)
- R pad 6: (no net) -> Net-(J4-Pad6)
- R pad 7: (no net) -> Net-(J4-Pad7)
- R pad 8: (no net) -> Net-(J4-Pad8)
Routing:
- net Net-(J2-Pad12): track 73.2 -> 0.00 mm
- net Net-(J2-Pad15): track 65.1 -> 127.7 mm
- net Net-(J2-Pad10): track 58.4 -> 0.00 mm
- net GND: track 110.0 -> 150.7 mm
- net Net-(J1-Pad2): track 27.6 -> 46.4 mm
- net Net-(J10-Pad1): track 82.1 -> 69.2 mm
- net Net-(J1-Pad7): track 37.4 -> 24.7 mm
- net Net-(J1-Pad13): track 36.3 -> 48.4 mm
- net Net-(J1-Pad1): track 25.4 -> 13.5 mm
- net Net-(J1-Pad8): track 28.8 -> 33.3 mm
- net Net-(D1-Pad2): track 33.3 -> 35.5 mm
- net +5V: track 54.0 -> 52.7 mm
- net Net-(J1-Pad5): track 26.2 -> 27.1 mm
- net Net-(J6-Pad1): track 16.3 -> 15.5 mm
- net Net-(D2-Pad1): track 15.1 -> 14.6 mm
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Other:
- board text added: "EMS-Receiver ICHINOSEKI"
- board text removed: "ICHINOSEKI-B EMS-Receiver 2021 Falco"

Commit message: Update Receiver.
Parts:
- removed 3.3V OUT: 3V3_OUT, Connector_JST:JST_XH_S2B-XH-A_1x02_P2.50mm_Horizontal
- removed CAN: CAN, Connector_JST:JST_XH_S2B-XH-A_1x02_P2.50mm_Horizontal
- removed I2C: I2C, Connector_JST:JST_XH_S2B-XH-A_1x02_P2.50mm_Horizontal
- removed L: F303k8_Left, Connector_PinSocket_2.54mm:PinSocket_1x15_P2.54mm_Vertical
- removed R: F303k8_Right, Connector_PinSocket_2.54mm:PinSocket_1x15_P2.54mm_Vertical
- removed the REF** at (159.0, 149.0)
- removed the REF** at (159.0, 95.0)
- removed the REF** at (85.0, 95.0)
- removed the REF** at (85.0, 149.0)
- added D3: LED, LED_THT:LED_D5.0mm, F.Cu at (141.0, 118.0)
- added D4: LED, LED_THT:LED_D5.0mm, F.Cu at (149.0, 118.0)
- added J1: RESS_OUT2, Connector_JST:JST_XH_S2B-XH-A_1x02_P2.50mm_Horizontal, F.Cu at (144.0, 131.0)
- added REF**: MountingHole_3.2mm_M3_Pad_Via, MountingHole:MountingHole_3.2mm_M3_Pad_Via, F.Cu at (149.0, 148.0)
- added REF**: MountingHole_3.2mm_M3_Pad_Via, MountingHole:MountingHole_3.2mm_M3_Pad_Via, F.Cu at (149.0, 109.0)
- added REF**: MountingHole_3.2mm_M3_Pad_Via, MountingHole:MountingHole_3.2mm_M3_Pad_Via, F.Cu at (85.0, 109.0)
- added REF**: MountingHole_3.2mm_M3_Pad_Via, MountingHole:MountingHole_3.2mm_M3_Pad_Via, F.Cu at (85.0, 148.0)
- added SW2: SW_SPDT, Connector_PinHeader_2.54mm:PinHeader_1x03_P2.54mm_Vertical, F.Cu at (145.0, 123.0)
- added U2: SeeeduinoXIAO, Seeeduino XIAO KICAD:Seeeduino XIAO-MOUDLE14P-2.54-21X17.8MM, F.Cu at (103.0, 131.0)
- added U3: LTV-817, Package_DIP:DIP-4_W7.62mm, F.Cu at (133.0, 137.0)
- J3: renamed from L; value ADP_Left -> ADP_L
- J4: renamed from R; value ADP_Right -> ADP_R
- J5: renamed from 5V IN
- J6: renamed from EMS; value EMS_OUT -> RESS_OUT1
- moved U1 34.1 mm to (86.0, 137.0)
- moved SW1 25.4 mm to (84.0, 123.0)
- moved D2 22.0 mm to (91.0, 118.5)
- moved J6 21.6 mm to (90.0, 128.5), turned to 270 degrees
- moved D1 13.6 mm to (84.0, 118.5)
- moved J3 12.0 mm to (99.4, 110.6)
- moved J4 12.0 mm to (124.8, 110.6)
- moved J5 11.4 mm to (108.0, 143.0)
- renumbered OFF to D1, ON to D2
Connections:
- J3 pad 1: Net-(J2-Pad15) -> (no net)
- J3 pad 10: Net-(J3-Pad10) -> (no net)
- J3 pad 2: Net-(J3-Pad2) -> (no net)
- J3 pad 3: Net-(J3-Pad3) -> (no net)
- J3 pad 4: Net-(J1-Pad2) -> RX
- J3 pad 5: Net-(J3-Pad5) -> (no net)
- J3 pad 6: Net-(J3-Pad6) -> (no net)
- J3 pad 7: Net-(J3-Pad7) -> (no net)
- J3 pad 8: Net-(J3-Pad8) -> (no net)
- J3 pad 9: Net-(J2-Pad14) -> +3V3
- J4 pad 1: Net-(J4-Pad1) -> (no net)
- J4 pad 10: Net-(J4-Pad10) -> (no net)
- J4 pad 2: Net-(J4-Pad2) -> (no net)
- J4 pad 3: Net-(J1-Pad1) -> TX
- J4 pad 4: Net-(J4-Pad4) -> (no net)
- J4 pad 5: Net-(J4-Pad5) -> (no net)
- J4 pad 6: Net-(J4-Pad6) -> (no net)
- J4 pad 7: Net-(J4-Pad7) -> (no net)
- J4 pad 8: Net-(J4-Pad8) -> (no net)
- U1 pad 1: Net-(J10-Pad1) -> Out1
Routing:
- net Net-(J2-Pad15): track 127.7 -> 0.00 mm
- net Out2: track 0.00 -> 71.4 mm, vias 0 -> 1
- net Net-(J10-Pad1): track 69.2 -> 0.00 mm
- net GND: track 150.7 -> 82.4 mm
- net Net-(J2-Pad14): track 57.3 -> 0.00 mm
- net Net-(J1-Pad13): track 48.4 -> 0.00 mm
- net Net-(J1-Pad2): track 46.4 -> 0.00 mm
- net Out1: track 0.00 -> 39.7 mm, vias 0 -> 1
- net RX: track 0.00 -> 36.9 mm, vias 0 -> 1
- net Net-(D2-Pad2): track 63.9 -> 27.7 mm
- net Net-(J1-Pad8): track 33.3 -> 0.00 mm
- net Net-(D4-Pad2): track 0.00 -> 31.9 mm
- net Net-(D3-Pad2): track 0.00 -> 29.1 mm
- net TX: track 0.00 -> 27.3 mm, vias 0 -> 1
- net Net-(J1-Pad5): track 27.1 -> 0.00 mm
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Other:
- board size 81.3 x 61 mm -> 72 x 47 mm
- board text removed: "EMS-Receiver ICHINOSEKI"
- board text removed: "OFF"
- board text removed: "ON"

Commit message: Modify the PCB and add the Gerber files.
Other:
- board text added: "RESS-Receiver 2022 Ichinoseki-B Falco"
Changed lines of the file:
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@@
   (general
     (thickness 1.6)
-    (drawings 4)
+    (drawings 5)
     (tracks 114)
     (zones 0)
@@
       (drillshape 0)
       (scaleselection 1)
-      (outputdirectory "../OutPut/Receiver/"))
+      (outputdirectory "Output/"))
   )
   (net 0 "")
@@
       (effects (font (size 1 1) (thickness 0.15)))
     )
+    (fp_circle (center 0 0) (end 3.2 0) (layer Cmts.User) (width 0.15))
+    (fp_circle (center 0 0) (end 3.45 0) (layer F.CrtYd) (width 0.05))
     (fp_text user %R (at 0.3 0) (layer F.Fab)
       (effects (font (size 1 1) (thickness 0.15)))
     )
-    (fp_circle (center 0 0) (end 3.2 0) (layer Cmts.User) (width 0.15))
-    (fp_circle (center 0 0) (end 3.45 0) (layer F.CrtYd) (width 0.05))
     (pad 1 thru_hole circle (at 1.697056 -1.697056) (size 0.8 0.8) (drill 0.5) (layers *.Cu *.Mask))
     (pad 1 thru_hole circle (at 0 -2.4) (size 0.8 0.8) (drill 0.5) (layers *.Cu *.Mask))
@@
       (effects (font (size 1 1) (thickness 0.15)))
     )
+    (fp_circle (center 0 0) (end 3.2 0) (layer Cmts.User) (width 0.15))
+    (fp_circle (center 0 0) (end 3.45 0) (layer F.CrtYd) (width 0.05))
     (fp_text user %R (at 0.3 0) (layer F.Fab)
       (effects (font (size 1 1) (thickness 0.15)))
     )
-    (fp_circle (center 0 0) (end 3.2 0) (layer Cmts.User) (width 0.15))
-    (fp_circle (center 0 0) (end 3.45 0) (layer F.CrtYd) (width 0.05))
     (pad 1 thru_hole circle (at 1.697056 -1.697056) (size 0.8 0.8) (drill 0.5) (layers *.Cu *.Mask))
     (pad 1 thru_hole circle (at 0 -2.4) (size 0.8 0.8) (drill 0.5) (layers *.Cu *.Mask))
@@
       (effects (font (size 1 1) (thickness 0.15)))
     )
+    (fp_circle (center 0 0) (end 3.2 0) (layer Cmts.User) (width 0.15))
+    (fp_circle (center 0 0) (end 3.45 0) (layer F.CrtYd) (width 0.05))
     (fp_text user %R (at 0.3 0) (layer F.Fab)
       (effects (font (size 1 1) (thickness 0.15)))
     )
-    (fp_circle (center 0 0) (end 3.2 0) (layer Cmts.User) (width 0.15))
-    (fp_circle (center 0 0) (end 3.45 0) (layer F.CrtYd) (width 0.05))
     (pad 1 thru_hole circle (at 1.697056 -1.697056) (size 0.8 0.8) (drill 0.5) (layers *.Cu *.Mask))
     (pad 1 thru_hole circle (at 0 -2.4) (size 0.8 0.8) (drill 0.5) (layers *.Cu *.Mask))
@@
       (effects (font (size 1 1) (thickness 0.15)))
     )
+    (fp_circle (center 0 0) (end 3.2 0) (layer Cmts.User) (width 0.15))
+    (fp_circle (center 0 0) (end 3.45 0) (layer F.CrtYd) (width 0.05))
     (fp_text user %R (at 0.3 0) (layer F.Fab)
       (effects (font (size 1 1) (thickness 0.15)))
     )
-    (fp_circle (center 0 0) (end 3.2 0) (layer Cmts.User) (width 0.15))
-    (fp_circle (center 0 0) (end 3.45 0) (layer F.CrtYd) (width 0.05))
     (pad 1 thru_hole circle (at 1.697056 -1.697056) (size 0.8 0.8) (drill 0.5) (layers *.Cu *.Mask))
     (pad 1 thru_hole circle (at 0 -2.4) (size 0.8 0.8) (drill 0.5) (layers *.Cu *.Mask))
@@
       (effects (font (size 1 1) (thickness 0.15)))
     )
-    (fp_text user %R (at 1.25 0 90) (layer F.Fab)
-      (effects (font (size 0.8 0.8) (thickness 0.2)))
-    )
-    (fp_arc (start 1.27 0) (end -1.29 1.54483) (angle -148.9) (layer F.SilkS) (width 0.12))
-    (fp_arc (start 1.27 0) (end -1.29 -1.54483) (angle 148.9) (layer F.SilkS) (width 0.12))
-    (fp_arc (start 1.27 0) (end -1.23 -1.469694) (angle 299.1) (layer F.Fab) (width 0.1))
     (fp_circle (center 1.27 0) (end 3.77 0) (layer F.Fab) (width 0.1))
     (fp_circle (center 1.27 0) (end 3.77 0) (layer F.SilkS) (width 0.12))
@@
     (fp_line (start 4.5 3.25) (end 4.5 -3.25) (layer F.CrtYd) (width 0.05))
     (fp_line (start 4.5 -3.25) (end -1.95 -3.25) (layer F.CrtYd) (width 0.05))
+    (fp_text user %R (at 1.25 0 90) (layer F.Fab)
+      (effects (font (size 0.8 0.8) (thickness 0.2)))
+    )
+    (fp_arc (start 1.27 0) (end -1.29 1.54483) (angle -148.9) (layer F.SilkS) (width 0.12))
+    (fp_arc (start 1.27 0) (end -1.29 -1.54483) (angle 148.9) (layer F.SilkS) (width 0.12))
+    (fp_arc (start 1.27 0) (end -1.23 -1.469694) (angle 299.1) (layer F.Fab) (width 0.1))
     (pad 2 thru_hole circle (at 2.54 0 90) (size 1.8 1.8) (drill 0.9) (layers *.Cu *.Mask)
       (net 12 "Net-(D3-Pad2)"))
@@
       (effects (font (size 1 1) (thickness 0.15)))
     )
-    (pad 1 thru_hole roundrect (at 0 0 90) (size 1.7 2) (drill 1) (layers *.Cu *.Mask) (roundrect_rratio 0.147059)
+    (pad 1 thru_hole roundrect (at 0 0 90) (size 1.7 2) (drill 1) (layers *.Cu *.Mask) (roundrect_rratio 0.1470588235294118)
       (net 5 "Net-(J1-Pad1)"))
     (pad 2 thru_hole oval (at 2.5 0 90) (size 1.7 2) (drill 1) (layers *.Cu *.Mask)
@@
     )
   )
+  (gr_text "RESS-Receiver\n2022 Ichinoseki-B\nFalco" (at 126 148) (layer F.SilkS)
+    (effects (font (size 1 1) (thickness 0.15)))
+  )
   (gr_line (start 153 105) (end 81 105) (layer Edge.Cuts) (width 0.05))
