File: RESS/Receiver/substrate/Receiver.sch (KiCad schematic (older format))
At the start: 17 parts, among them J3 ADP_L, J4 ADP_R, J5 Power, J6 RESS_OUT1, SW1 SW_SPDT, SW2 SW_DIP_x02, U1 LTV-817, U2 RR-1A, U3 TA48033S, U4 TC74HC32AP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

Commit message: P10を3.3Vと接続するのを忘れていたので修正
Parts:
- D1, D2: symbol Receiver-rescue:LED-Device-Receiver-rescue-Receiver-rescue-Receiver-rescue -> Receiver-rescue:LED-Device-Receiver-rescue-Receiver-rescue-Receiver-rescue-Receiver-rescue
- J3, J4: symbol Receiver-rescue:Conn_01x10_Female-Connector-Receiver-rescue-Receiver-rescue-Receiver-rescue -> Receiver-rescue:Conn_01x10_Female-Connector-Receiver-rescue-Receiver-rescue-Receiver-rescue-Receiver-rescue
- J5, J6: symbol Receiver-rescue:Conn_01x02_Male-Connector-Receiver-rescue-Receiver-rescue-Receiver-rescue -> Receiver-rescue:Conn_01x02_Male-Connector-Receiver-rescue-Receiver-rescue-Receiver-rescue-Receiver-rescue
- SW1: symbol Receiver-rescue:SW_SPDT-Switch-Receiver-rescue-Receiver-rescue-Receiver-rescue -> Receiver-rescue:SW_SPDT-Switch-Receiver-rescue-Receiver-rescue-Receiver-rescue-Receiver-rescue
- U1: symbol Receiver-rescue:LTV-817-Isolator-Receiver-rescue-Receiver-rescue-Receiver-rescue -> Receiver-rescue:LTV-817-Isolator-Receiver-rescue-Receiver-rescue-Receiver-rescue-Receiver-rescue
- U2: symbol Receiver-rescue:RR-1A-RR-1A -> Receiver-rescue:RR-1A-RR-1A-Receiver-rescue
- U4: symbol 74:TC74HC32AP -> Receiver-rescue:TC74HC32AP-74
- U5: symbol 74:TC74HC08AP -> Receiver-rescue:TC74HC08AP-74
Connections:
- net +3V3: now also J4.5 (Pin_5)
Changed lines of the file:
@@
 $EndDescr
 $Comp
-L Receiver-rescue:GND-power-Receiver-rescue-Receiver-rescue-Receiver-rescue #PWR0101
+L Receiver-rescue:GND-power-Receiver-rescue-Receiver-rescue-Receiver-rescue-Receiver-rescue #PWR0101
 U 1 1 60AF1801
 P 6500 4400
@@
 $EndComp
 $Comp
-L Receiver-rescue:Conn_01x02_Male-Connector-Receiver-rescue-Receiver-rescue-Receiver-rescue J5
+L Receiver-rescue:Conn_01x02_Male-Connector-Receiver-rescue-Receiver-rescue-Receiver-rescue-Receiver-rescue J5
 U 1 1 60B39C1D
 P 6250 4300
@@
 $EndComp
 $Comp
-L Receiver-rescue:LTV-817-Isolator-Receiver-rescue-Receiver-rescue-Receiver-rescue U1
+L Receiver-rescue:LTV-817-Isolator-Receiver-rescue-Receiver-rescue-Receiver-rescue-Receiver-rescue U1
 U 1 1 60AF1260
 P 5500 4350
@@
 $EndComp
 $Comp
-L Receiver-rescue:LED-Device-Receiver-rescue-Receiver-rescue-Receiver-rescue D1
+L Receiver-rescue:LED-Device-Receiver-rescue-Receiver-rescue-Receiver-rescue-Receiver-rescue D1
 U 1 1 60B360E0
 P 5800 4700
@@
 $EndComp
 $Comp
-L Receiver-rescue:SW_SPDT-Switch-Receiver-rescue-Receiver-rescue-Receiver-rescue SW1
+L Receiver-rescue:SW_SPDT-Switch-Receiver-rescue-Receiver-rescue-Receiver-rescue-Receiver-rescue SW1
 U 1 1 60B49C25
 P 6250 4800
@@
 	5600 4700 5650 4700
 $Comp
-L Receiver-rescue:LED-Device-Receiver-rescue-Receiver-rescue-Receiver-rescue D2
+L Receiver-rescue:LED-Device-Receiver-rescue-Receiver-rescue-Receiver-rescue-Receiver-rescue D2
 U 1 1 60B97B28
 P 5800 4900
@@
 	5650 4900 5400 4900
 $Comp
-L Receiver-rescue:+5V-power-Receiver-rescue-Receiver-rescue-Receiver-rescue #PWR0104
+L Receiver-rescue:+5V-power-Receiver-rescue-Receiver-rescue-Receiver-rescue-Receiver-rescue #PWR0104
 U 1 1 60B5796E
 P 6500 4300
@@
 NoConn ~ 6600 3950
 NoConn ~ 6600 3750
-NoConn ~ 6600 3450
 NoConn ~ 6600 3350
 NoConn ~ 6600 3150
 NoConn ~ 6150 3150
 NoConn ~ 6150 3250
-NoConn ~ 6150 3450
 NoConn ~ 6150 3750
 NoConn ~ 6150 3950
@@
 NoConn ~ 6150 3650
 $Comp
-L Receiver-rescue:Conn_01x10_Female-Connector-Receiver-rescue-Receiver-rescue-Receiver-rescue J4
+L Receiver-rescue:Conn_01x10_Female-Connector-Receiver-rescue-Receiver-rescue-Receiver-rescue-Receiver-rescue J4
 U 1 1 60B038BF
 P 6400 3450
@@
 $EndComp
 $Comp
-L Receiver-rescue:Conn_01x10_Female-Connector-Receiver-rescue-Receiver-rescue-Receiver-rescue J3
+L Receiver-rescue:Conn_01x10_Female-Connector-Receiver-rescue-Receiver-rescue-Receiver-rescue-Receiver-rescue J3
 U 1 1 60B01E56
 P 6350 3450
@@
 	6450 4800 6550 4800
 $Comp
-L Receiver-rescue:Conn_01x02_Male-Connector-Receiver-rescue-Receiver-rescue-Receiver-rescue J6
+L Receiver-rescue:Conn_01x02_Male-Connector-Receiver-rescue-Receiver-rescue-Receiver-rescue-Receiver-rescue J6
 U 1 1 60BC7FBD
 P 6750 4800
@@
 	8100 2850 8100 5100
 $Comp
-L Receiver-rescue:RR-1A-RR-1A U2
+L Receiver-rescue:RR-1A-RR-1A-Receiver-rescue U2
 U 1 1 62C7EF96
 P 4400 3200
@@
 DIP-SW
 $Comp
-L 74:TC74HC32AP U4
+L Receiver-rescue:TC74HC32AP-74 U4
 U 1 1 62CAEDC7
 P 7550 3450
@@
 OUT6
 $Comp
-L 74:TC74HC08AP U5
+L Receiver-rescue:TC74HC08AP-74 U5
 U 1 1 62CBA817
 P 7550 4550
@@
 	1    0    0    -1
 $EndComp
+NoConn ~ 6150 3450
+$Comp
+L power:+3.3V #PWR?
+U 1 1 62C83FA5
+P 6700 3400
+F 0 "#PWR?" H 6700 3250 50  0001 C CNN
+F 1 "+3.3V" H 6750 3550 50  0000 C CNN
+F 2 "" H 6700 3400 50  0001 C CNN
+F 3 "" H 6700 3400 50  0001 C CNN
+	1    6700 3400
+	1    0    0    -1
+$EndComp
+NoConn ~ 6600 3250
+Wire Wire Line
+	6600 3450 6700 3450
+Wire Wire Line
+	6700 3450 6700 3400
 $EndSCHEMATC

Commit message: 回路の細かな修正
Parts:
- D1, D2: symbol Receiver-rescue:LED-Device-Receiver-rescue-Receiver-rescue-Receiver-rescue-Receiver-rescue -> Receiver-rescue:LED-Device-Receiver-rescue-Receiver-rescue-Receiver-rescue-Receiver-rescue-Receiver-rescue
- J3, J4: symbol Receiver-rescue:Conn_01x10_Female-Connector-Receiver-rescue-Receiver-rescue-Receiver-rescue-Receiver-rescue -> Receiver-rescue:Conn_01x10_Female-Connector-Receiver-rescue-Receiver-rescue-Receiver-rescue-Receiver-rescue-Receiver-re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
- J5, J6: symbol Receiver-rescue:Conn_01x02_Male-Connector-Receiver-rescue-Receiver-rescue-Receiver-rescue-Receiver-rescue -> Receiver-rescue:Conn_01x02_Male-Connector-Receiver-rescue-Receiver-rescue-Receiver-rescue-Receiver-rescue-Receiver-resc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
- SW1: symbol Receiver-rescue:SW_SPDT-Switch-Receiver-rescue-Receiver-rescue-Receiver-rescue-Receiver-rescue -> Receiver-rescue:SW_SPDT-Switch-Receiver-rescue-Receiver-rescue-Receiver-rescue-Receiver-rescue-Receiver-rescue
- U1: symbol Receiver-rescue:LTV-817-Isolator-Receiver-rescue-Receiver-rescue-Receiver-rescue-Receiver-rescue -> Receiver-rescue:LTV-817-Isolator-Receiver-rescue-Receiver-rescue-Receiver-rescue-Receiver-rescue-Receiver-rescue
- U2: symbol Receiver-rescue:RR-1A-RR-1A-Receiver-rescue -> Receiver-rescue:RR-1A-RR-1A-Receiver-rescue-Receiver-rescue
- U4: symbol Receiver-rescue:TC74HC32AP-74 -> Receiver-rescue:TC74HC32AP-74-Receiver-rescue
- U5: symbol Receiver-rescue:TC74HC08AP-74 -> Receiver-rescue:TC74HC08AP-74-Receiver-rescue
Changed lines of the file:
@@
 $EndDescr
 $Comp
-L Receiver-rescue:GND-power-Receiver-rescue-Receiver-rescue-Receiver-rescue-Receiver-rescue #PWR0101
+L Receiver-rescue:GND-power-Receiver-rescue-Receiver-rescue-Receiver-rescue-Receiver-rescue-Receiver-rescue #PWR0101
 U 1 1 60AF1801
 P 6500 4400
@@
 $EndComp
 $Comp
-L Receiver-rescue:Conn_01x02_Male-Connector-Receiver-rescue-Receiver-rescue-Receiver-rescue-Receiver-rescue J5
+L Receiver-rescue:Conn_01x02_Male-Connector-Receiver-rescue-Receiver-rescue-Receiver-rescue-Receiver-rescue-Receiver-rescue J5
 U 1 1 60B39C1D
 P 6250 4300
@@
 $EndComp
 $Comp
-L Receiver-rescue:LTV-817-Isolator-Receiver-rescue-Receiver-rescue-Receiver-rescue-Receiver-rescue U1
+L Receiver-rescue:LTV-817-Isolator-Receiver-rescue-Receiver-rescue-Receiver-rescue-Receiver-rescue-Receiver-rescue U1
 U 1 1 60AF1260
 P 5500 4350
@@
 $EndComp
 $Comp
-L Receiver-rescue:LED-Device-Receiver-rescue-Receiver-rescue-Receiver-rescue-Receiver-rescue D1
+L Receiver-rescue:LED-Device-Receiver-rescue-Receiver-rescue-Receiver-rescue-Receiver-rescue-Receiver-rescue D1
 U 1 1 60B360E0
 P 5800 4700
@@
 $EndComp
 $Comp
-L Receiver-rescue:SW_SPDT-Switch-Receiver-rescue-Receiver-rescue-Receiver-rescue-Receiver-rescue SW1
+L Receiver-rescue:SW_SPDT-Switch-Receiver-rescue-Receiver-rescue-Receiver-rescue-Receiver-rescue-Receiver-rescue SW1
 U 1 1 60B49C25
 P 6250 4800
@@
 	5600 4700 5650 4700
 $Comp
-L Receiver-rescue:LED-Device-Receiver-rescue-Receiver-rescue-Receiver-rescue-Receiver-rescue D2
+L Receiver-rescue:LED-Device-Receiver-rescue-Receiver-rescue-Receiver-rescue-Receiver-rescue-Receiver-rescue D2
 U 1 1 60B97B28
 P 5800 4900
@@
 	5650 4900 5400 4900
 $Comp
-L Receiver-rescue:+5V-power-Receiver-rescue-Receiver-rescue-Receiver-rescue-Receiver-rescue #PWR0104
+L Receiver-rescue:+5V-power-Receiver-rescue-Receiver-rescue-Receiver-rescue-Receiver-rescue-Receiver-rescue #PWR0104
 U 1 1 60B5796E
 P 6500 4300
@@
 NoConn ~ 6150 3650
 $Comp
-L Receiver-rescue:Conn_01x10_Female-Connector-Receiver-rescue-Receiver-rescue-Receiver-rescue-Receiver-rescue J4
+L Receiver-rescue:Conn_01x10_Female-Connector-Receiver-rescue-Receiver-rescue-Receiver-rescue-Receiver-rescue-Receiver-rescue J4
 U 1 1 60B038BF
 P 6400 3450
@@
 $EndComp
 $Comp
-L Receiver-rescue:Conn_01x10_Female-Connector-Receiver-rescue-Receiver-rescue-Receiver-rescue-Receiver-rescue J3
+L Receiver-rescue:Conn_01x10_Female-Connector-Receiver-rescue-Receiver-rescue-Receiver-rescue-Receiver-rescue-Receiver-rescue J3
 U 1 1 60B01E56
 P 6350 3450
@@
 	6450 4800 6550 4800
 $Comp
-L Receiver-rescue:Conn_01x02_Male-Connector-Receiver-rescue-Receiver-rescue-Receiver-rescue-Receiver-rescue J6
+L Receiver-rescue:Conn_01x02_Male-Connector-Receiver-rescue-Receiver-rescue-Receiver-rescue-Receiver-rescue-Receiver-rescue J6
 U 1 1 60BC7FBD
 P 6750 4800
@@
 	8100 2850 8100 5100
 $Comp
-L Receiver-rescue:RR-1A-RR-1A-Receiver-rescue U2
+L Receiver-rescue:RR-1A-RR-1A-Receiver-rescue-Receiver-rescue U2
 U 1 1 62C7EF96
 P 4400 3200
@@
 DIP-SW
 $Comp
-L Receiver-rescue:TC74HC32AP-74 U4
+L Receiver-rescue:TC74HC32AP-74-Receiver-rescue U4
 U 1 1 62CAEDC7
 P 7550 3450
@@
 OUT6
 $Comp
-L Receiver-rescue:TC74HC08AP-74 U5
+L Receiver-rescue:TC74HC08AP-74-Receiver-rescue U5
 U 1 1 62CBA817
 P 7550 4550

Commit message: 基板が燃えるほどのミスを修正
Parts:
- removed U1: LTV-817, Package_DIP:DIP-4_W7.62mm, symbol Receiver-rescue:LTV-817-Isolator-Receiver-rescue-Receiver-rescue-Receiver-rescu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
- removed U3: TA48033S, Package_TO_SOT_THT:TO-220-3_Horizontal_TabDown, symbol MyComponent:TA48033S
- added C1: 0.33μF, Capacitor_THT:C_Rect_L4.0mm_W2.5mm_P2.50mm, symbol Device:C
- added C2: 47μF, Capacitor_THT:CP_Radial_D5.0mm_P2.00mm, symbol Device:CP
- added R1: 220Ω, Resistor_THT:R_Axial_DIN0207_L6.3mm_D2.5mm_P7.62mm_Horizontal, symbol Device:R
- added U1: TLP785, Package_DIP:DIP-4_W7.62mm, symbol Isolator:TLP785
- added U3: 48033S, Package_TO_SOT_THT:TO-220-3_Horizontal_TabDown, symbol Regulator_Linear:AP2204R-3.3
- D1, D2: symbol Receiver-rescue:LED-Device-Receiver-rescue-Receiver-rescue-Receiver-rescue-Receiver-rescue-Receiver-rescue -> Receiver-rescue:LED-Device-Receiver-rescue-Receiver-rescue-Receiver-rescue-Receiver-rescue-Receiver-rescue-Receiver-res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
- J3, J4: symbol Receiver-rescue:Conn_01x10_Female-Connector-Receiver-rescue-Receiver-rescue-Receiver-rescue-Receiver-rescue-Receiver-rescue -> Receiver-rescue:Conn_01x10_Female-Connector-Receiver-rescue-Receiver-rescue-Receiver-rescue-Receiver-rescue-Receiver-rescue-Receiver-rescue-Receiver-rescue
- J5, J6: symbol Receiver-rescue:Conn_01x02_Male-Connector-Receiver-rescue-Receiver-rescue-Receiver-rescue-Receiver-rescue-Receiver-rescue -> Receiver-rescue:Conn_01x02_Male-Connector-Receiver-rescue-Receiver-rescue-Receiver-rescue-Receiver-rescue-Receiver-rescue-Receiver-rescue-Receiver-rescue
- SW1: symbol Receiver-rescue:SW_SPDT-Switch-Receiver-rescue-Receiver-rescue-Receiver-rescue-Receiver-rescue-Receiver-rescue -> Receiver-rescue:SW_SPDT-Switch-Receiver-rescue-Receiver-rescue-Receiver-rescue-Receiver-rescue-Receiver-rescue-Receiver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
- U2: symbol Receiver-rescue:RR-1A-RR-1A-Receiver-rescue-Receiver-rescue -> Receiver-rescue:RR-1A-RR-1A-Receiver-rescue-Receiver-rescue-Receiver-rescue-Receiver-rescue
- U4: symbol Receiver-rescue:TC74HC32AP-74-Receiver-rescue -> Receiver-rescue:TC74HC32AP-74-Receiver-rescue-Receiver-rescue-Receiver-rescue
- U5: symbol Receiver-rescue:TC74HC08AP-74-Receiver-rescue -> Receiver-rescue:TC74HC08AP-74-Receiver-rescue-Receiver-rescue-Receiver-rescue
Connections:
- net +3V3: now also C2.1, U3.3 (VOUT)
- net +5V: now also C1.1, U3.1 (VIN)
- net GND: now also C1.2, C2.2, U1.2, U3.2 (GND)
- net OUT: now also R1.2
- net at D1.2 (A): now also SW1.1 (A)
- net at D2.2 (A): now also SW1.3 (C); no longer J6.2 (Pin_2)
- net at D1.1 (K): now also U1.4; no longer SW1.1 (A)
- net at D2.1 (K): now also J6.2 (Pin_2), U1.3; no longer SW1.3 (C)
- new net: R1.1, U1.1
Other:
- moved on the sheet: D1, D2, J6, SW1, SW2
