File: RESS/Transmitter/substrate/Transmitter.sch (KiCad schematic (older format))
At the start: 9 parts, among them J3 ADP_L, J4 ADP_R, J5 POWER, J6 ESS_IN, SW1 SW_SPDT, U1 SeeeduinoXIAO

Commit message: 送信基板の追加とファイルの整理
Parts:
- removed U1: SeeeduinoXIAO, Seeeduino XIAO KICAD:Seeeduino XIAO-MOUDLE14P-2.54-21X17.8MM, symbol Seeeduino_XIAO:SeeeduinoXIAO
- added D1: LED, LED_THT:LED_D5.0mm, symbol Device:LED
- added H1, H2, H3, H4: MountingHole, MountingHole:MountingHole_3.2mm_M3_Pad_Via, symbol Mechanical:MountingHole
- added R4: 10kΩ, Resistor_THT:R_Axial_DIN0207_L6.3mm_D2.5mm_P7.62mm_Horizontal, symbol Device:R
- J3, J4: symbol Transmitter-rescue:Conn_01x10_Female-Connector-Transmitter-rescue-Transmitter-rescue -> Transmitter-rescue:Conn_01x10_Female-Connector-Transmitter-rescue-Transmitter-rescue-Transmitter-rescue
- J5, J6: symbol Transmitter-rescue:Conn_01x02_Male-Connector-Transmitter-rescue-Transmitter-rescue -> Transmitter-rescue:Conn_01x02_Male-Connector-Transmitter-rescue-Transmitter-rescue-Transmitter-rescue
- SW1: symbol Transmitter-rescue:SW_SPDT-Switch-Transmitter-rescue-Transmitter-rescue -> Transmitter-rescue:SW_SPDT-Switch-Transmitter-rescue-Transmitter-rescue-Transmitter-rescue
Connections:
- net +3V3: now also J3.5 (Pin_5)
- net GND: now also J4.1 (Pin_1), D1.1 (K), R4.1
- net ESS_IN renamed LED
- net LED: now also D1.2 (A), R4.2
- net RX: no longer names the net of J3.4 (Pin_4)
- net TX: no longer names the net of J4.3 (Pin_3)
- no-connect marks 31 -> 17
Other:
- note added: "Hole"
- note added: "LED"
- note removed: "RTS"
- note removed: "RxD"
- note removed: "SeeeduinoXIAO"
- note removed: "TxD"
- moved on the sheet: J3, J4, J5, J6, R1, R2, R3, SW1

Commit message: 回路の細かな修正
Parts:
- added U1: TA48033S, Package_TO_SOT_THT:TO-220-3_Horizontal_TabDown, symbol MyComponent:TA48033S
- J3, J4: symbol Transmitter-rescue:Conn_01x10_Female-Connector-Transmitter-rescue-Transmitter-rescue-Transmitter-rescue -> Transmitter-rescue:Conn_01x10_Female-Connector-Transmitter-rescue-Transmitter-rescue-Transmitter-rescue-Transmitter-res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
- J5, J6: symbol Transmitter-rescue:Conn_01x02_Male-Connector-Transmitter-rescue-Transmitter-rescue-Transmitter-rescue -> Transmitter-rescue:Conn_01x02_Male-Connector-Transmitter-rescue-Transmitter-rescue-Transmitter-rescue-Transmitter-rescu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
- SW1: symbol Transmitter-rescue:SW_SPDT-Switch-Transmitter-rescue-Transmitter-rescue-Transmitter-rescue -> Transmitter-rescue:SW_SPDT-Switch-Transmitter-rescue-Transmitter-rescue-Transmitter-rescue-Transmitter-rescue-Transmitt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
Connections:
- net +3V3: now also U1.2 (Vout)
- net +5V: now also U1.1 (Vin)
- net GND: now also U1.3 (GND)
Other:
- note added: "Regulator"
- moved on the sheet: J5
Changed lines of the file:
@@
 $EndDescr
 $Comp
-L Transmitter-rescue:Conn_01x10_Female-Connector-Transmitter-rescue-Transmitter-rescue-Transmitter-rescue J3
+L Transmitter-rescue:Conn_01x10_Female-Connector-Transmitter-rescue-Transmitter-rescue-Transmitter-rescue-Transmitter-rescue-Transmitter-rescue J3
 U 1 1 60B0F59A
 P 6300 3350
@@
 $EndComp
 $Comp
-L Transmitter-rescue:Conn_01x10_Female-Connector-Transmitter-rescue-Transmitter-rescue-Transmitter-rescue J4
+L Transmitter-rescue:Conn_01x10_Female-Connector-Transmitter-rescue-Transmitter-rescue-Transmitter-rescue-Transmitter-rescue-Transmitter-rescue J4
 U 1 1 60B10C64
 P 6400 3350
@@
 NoConn ~ 6600 3850
 $Comp
-L Transmitter-rescue:Conn_01x02_Male-Connector-Transmitter-rescue-Transmitter-rescue-Transmitter-rescue J5
+L Transmitter-rescue:Conn_01x02_Male-Connector-Transmitter-rescue-Transmitter-rescue-Transmitter-rescue-Transmitter-rescue-Transmitter-rescue J5
 U 1 1 60C2BF9E
-P 4350 3250
-F 0 "J5" H 4458 3431 50  0000 C CNN
-F 1 "POWER" H 4458 3340 50  0000 C CNN
-F 2 "Connector_JST:JST_XH_S2B-XH-A_1x02_P2.50mm_Horizontal" H 4350 3250 50  0001 C CNN
-F 3 "~" H 4350 3250 50  0001 C CNN
-	1    4350 3250
-	1    0    0    -1
-$EndComp
-$Comp
-L Transmitter-rescue:+5V-power-Transmitter-rescue-Transmitter-rescue-Transmitter-rescue #PWR01
+P 4350 3200
+F 0 "J5" H 4458 3381 50  0000 C CNN
+F 1 "POWER" H 4458 3290 50  0000 C CNN
+F 2 "Connector_JST:JST_XH_S2B-XH-A_1x02_P2.50mm_Horizontal" H 4350 3200 50  0001 C CNN
+F 3 "~" H 4350 3200 50  0001 C CNN
+	1    4350 3200
+	1    0    0    -1
+$EndComp
+$Comp
+L Transmitter-rescue:+5V-power-Transmitter-rescue-Transmitter-rescue-Transmitter-rescue-Transmitter-rescue-Transmitter-rescue #PWR01
 U 1 1 60C2C475
 P 5800 3100
@@
 $EndComp
 $Comp
-L Transmitter-rescue:GND-power-Transmitter-rescue-Transmitter-rescue-Transmitter-rescue #PWR02
+L Transmitter-rescue:GND-power-Transmitter-rescue-Transmitter-rescue-Transmitter-rescue-Transmitter-rescue-Transmitter-rescue #PWR02
 U 1 1 60C2CC2C
-P 4650 3450
-F 0 "#PWR02" H 4650 3200 50  0001 C CNN
-F 1 "GND" H 4500 3400 50  0000 C CNN
-F 2 "" H 4650 3450 50  0001 C CNN
-F 3 "" H 4650 3450 50  0001 C CNN
-	1    4650 3450
+P 4650 3400
+F 0 "#PWR02" H 4650 3150 50  0001 C CNN
+F 1 "GND" H 4500 3350 50  0000 C CNN
+F 2 "" H 4650 3400 50  0001 C CNN
+F 3 "" H 4650 3400 50  0001 C CNN
+	1    4650 3400
 	1    0    0    -1
 $EndComp
@@
 	5800 3250 5800 3100
 Wire Wire Line
-	4550 3350 4650 3350
-$Comp
-L Transmitter-rescue:Conn_01x02_Male-Connector-Transmitter-rescue-Transmitter-rescue-Transmitter-rescue J6
+	4550 3300 4650 3300
+$Comp
+L Transmitter-rescue:Conn_01x02_Male-Connector-Transmitter-rescue-Transmitter-rescue-Transmitter-rescue-Transmitter-rescue-Transmitter-rescue J6
 U 1 1 60B16252
 P 3200 3000
@@
 $EndComp
 $Comp
-L Transmitter-rescue:SW_SPDT-Switch-Transmitter-rescue-Transmitter-rescue-Transmitter-rescue SW1
+L Transmitter-rescue:SW_SPDT-Switch-Transmitter-rescue-Transmitter-rescue-Transmitter-rescue-Transmitter-rescue-Transmitter-rescue SW1
 U 1 1 60B2577F
 P 5500 3350
@@
 	3500 3000 3500 2950
 NoConn ~ 5700 3450
-Text GLabel 4650 3250 2    50   Input ~ 0
+Text GLabel 4650 3200 2    50   Input ~ 0
 PW_IN
 Wire Wire Line
-	4550 3250 4650 3250
-Wire Wire Line
-	4650 3350 4650 3450
+	4550 3200 4650 3200
+Wire Wire Line
+	4650 3300 4650 3400
 Text GLabel 5250 3350 0    50   Input ~ 0
 PW_IN
@@
 Text Notes 3150 2900 0    50   ~ 0
 ESS
-Text Notes 4700 3050 0    50   ~ 0
+Text Notes 4300 2900 0    50   ~ 0
 Power
 Text Notes 5000 2900 0    50   ~ 0
@@
 	5850 3550 4950 3550
 Wire Notes Line
-	3100 2800 6800 2800
-Wire Notes Line
 	3100 4250 6800 4250
 Wire Notes Line
@@
 Hole
 Wire Notes Line
-	3100 4600 6800 4600
-Wire Notes Line
 	3100 2800 3100 4600
 Wire Notes Line
 	6800 2800 6800 4600
+$Comp
+L MyComponent:TA48033S U1
+U 1 1 62C9172D
+P 7300 3550
+F 0 "U1" H 7300 3915 50  0000 C CNN
+F 1 "TA48033S" H 7300 3824 50  0000 C CNN
+F 2 "Package_TO_SOT_THT:TO-220-3_Horizontal_TabDown" H 7300 3850 50  0001 C CNN
+F 3 "" H 7300 3850 50  0001 C CNN
+	1    7300 3550
+	1    0    0    -1
+$EndComp
+$Comp
+L power:+3.3V #PWR0105
+U 1 1 62C935D3
+P 7700 3400
+F 0 "#PWR0105" H 7700 3250 50  0001 C CNN
+F 1 "+3.3V" H 7715 3573 50  0000 C CNN
+F 2 "" H 7700 3400 50  0001 C CNN
+F 3 "" H 7700 3400 50  0001 C CNN
+	1    7700 3400
+	1    0    0    -1
+$EndComp
+$Comp
+L power:+5V #PWR0109
+U 1 1 62C93BBD
+P 6900 3400
+F 0 "#PWR0109" H 6900 3250 50  0001 C CNN
+F 1 "+5V" H 6915 3573 50  0000 C CNN
+F 2 "" H 6900 3400 50  0001 C CNN
+F 3 "" H 6900 3400 50  0001 C CNN
+	1    6900 3400
+	1    0    0    -1
+$EndComp
+$Comp
+L power:GND #PWR0110
+U 1 1 62C93FAE
+P 7300 3800
+F 0 "#PWR0110" H 7300 3550 50  0001 C CNN
+F 1 "GND" H 7305 3627 50  0000 C CNN
+F 2 "" H 7300 3800 50  0001 C CNN
+F 3 "" H 7300 3800 50  0001 C CNN
+	1    7300 3800
+	1    0    0    -1
+$EndComp
+Wire Wire Line
+	6900 3400 6900 3450
+Wire Wire Line
+	6900 3450 6950 3450
+Wire Wire Line
+	7650 3450 7700 3450
+Wire Wire Line
+	7700 3450 7700 3400
+Wire Wire Line
+	7300 3750 7300 3800
+Wire Notes Line
+	7850 2800 7850 4600
+Wire Notes Line
+	3100 2800 7850 2800
+Wire Notes Line
+	3100 4600 7850 4600
+Text Notes 6850 2900 0    50   ~ 0
+Regulator
 $EndSCHEMATC

Commit message: 基板が燃えるほどのミスを修正
Parts:
- removed U1: TA48033S, Package_TO_SOT_THT:TO-220-3_Horizontal_TabDown, symbol MyComponent:TA48033S
- added C1: 0.33μF, Capacitor_THT:C_Rect_L4.0mm_W2.5mm_P2.50mm, symbol Device:C
- added C2: 47μF, Capacitor_THT:CP_Radial_D5.0mm_P2.00mm, symbol Device:CP
- added U1: BP5293, Package_TO_SOT_THT:TO-220-3_Horizontal_TabDown, symbol Regulator_Linear:AP2204R-3.0
- added U2: TLP785, Package_DIP:DIP-4_W7.62mm, symbol Isolator:TLP785
- J3, J4: symbol Transmitter-rescue:Conn_01x10_Female-Connector-Transmitter-rescue-Transmitter-rescue-Transmitter-rescue-Transmitter-rescue-Transmitter-rescue -> Transmitter-rescue:Conn_01x10_Female-Connector-Transmitter-rescue-Transmitter-rescue-Transmitter-rescue-Transmitter-rescue-Transmitter-rescue-Transmitter-rescue-Transmitter-rescue
- J5, J6: symbol Transmitter-rescue:Conn_01x02_Male-Connector-Transmitter-rescue-Transmitter-rescue-Transmitter-rescue-Transmitter-rescue-Transmitter-rescue -> Transmitter-rescue:Conn_01x02_Male-Connector-Transmitter-rescue-Transmitter-rescue-Transmitter-rescue-Transmitter-rescue-Transmitter-rescue-Transmitter-rescue-Transmitter-rescue
- R1, R2, R3: value 18Ω -> 22Ω
- R4: value 10kΩ -> 220Ω
- SW1: symbol Transmitter-rescue:SW_SPDT-Switch-Transmitter-rescue-Transmitter-rescue-Transmitter-rescue-Transmitter-rescue-Transmitter-rescue -> Transmitter-rescue:SW_SPDT-Switch-Transmitter-rescue-Transmitter-rescue-Transmitter-rescue-Transmitter-rescue-Transmitter-rescue-Transmitter-rescue-Transmitter-rescue
Connections:
- net +3V3: now also C2.1, U1.3 (VOUT), U2.4
- net +5V: now also C1.1, U1.1 (VIN)
- net GND: now also C1.2, C2.2, U1.2 (GND), U2.2; no longer J4.1 (Pin_1), R4.1
- new net: R4.1, U2.1
- new net ESS: J4.1 (Pin_1), U2.3
Other:
- moved on the sheet: J5, J6
