File: RESS-920/Receiver/circuit/Receiver.sch (KiCad schematic (older format))
At the start: 13 parts, among them J3 ADP_L, J4 ADP_R, J5 Power_IN, J6 RESS_OUT1, SW1 SW_SPDT, U1 LTV-817, U2 SeeeduinoXIAO

Commit message: WIP
Connections:
- net Out1 renamed Out
- net Out2: no longer names the net of U2.4 (PA11_A3_D3)
- no-connect marks 29 -> 30
Changed lines of the file:
@@
 	6950 3600 6950 3650
 Text GLabel 4050 3450 0    50   Input ~ 0
-Out1
+Out
 Wire Wire Line
 	4050 3450 4150 3450
 Text GLabel 6550 3600 0    50   Input ~ 0
-Out1
+Out
 Wire Wire Line
 	6550 3600 6600 3600
@@
 NoConn ~ 4150 3150
 NoConn ~ 4150 3300
-Text GLabel 4050 3600 0    50   Input ~ 0
-Out2
-Wire Wire Line
-	4050 3600 4150 3600
 Wire Wire Line
 	6600 4500 6600 4650
@@
 Text Notes 8150 2550 0    50   ~ 0
 MountingHole
+NoConn ~ 4150 3600
 $EndSCHEMATC
