File: RESS-920/Transmitter/circuit/Transmitter.sch (KiCad schematic (older format))
At the start: 9 parts, among them J3 ADP_L, J4 ADP_R, J5 POWER, J6 ESS_IN, SW1 SW_SPDT, U1 SeeeduinoXIAO

Commit message: WIP
Parts:
- J3, J4: symbol Transmitter-rescue:Conn_01x10_Female-Connector-Transmitter-rescue-Transmitter-rescue -> Transmitter-rescue:Conn_01x10_Female-Connector-Transmitter-rescue-Transmitter-rescue-Transmitter-rescue
- J5, J6: symbol Transmitter-rescue:Conn_01x02_Male-Connector-Transmitter-rescue-Transmitter-rescue -> Transmitter-rescue:Conn_01x02_Male-Connector-Transmitter-rescue-Transmitter-rescue-Transmitter-rescue
- SW1: symbol Transmitter-rescue:SW_SPDT-Switch-Transmitter-rescue-Transmitter-rescue -> Transmitter-rescue:SW_SPDT-Switch-Transmitter-rescue-Transmitter-rescue-Transmitter-rescue
Changed lines of the file:
@@
 $EndDescr
 $Comp
-L Transmitter-rescue:Conn_01x10_Female-Connector-Transmitter-rescue-Transmitter-rescue J3
+L Transmitter-rescue:Conn_01x10_Female-Connector-Transmitter-rescue-Transmitter-rescue-Transmitter-rescue J3
 U 1 1 60B0F59A
 P 6600 3850
@@
 $EndComp
 $Comp
-L Transmitter-rescue:Conn_01x10_Female-Connector-Transmitter-rescue-Transmitter-rescue J4
+L Transmitter-rescue:Conn_01x10_Female-Connector-Transmitter-rescue-Transmitter-rescue-Transmitter-rescue J4
 U 1 1 60B10C64
 P 6700 3850
@@
 NoConn ~ 6900 4350
 $Comp
-L Transmitter-rescue:Conn_01x02_Male-Connector-Transmitter-rescue-Transmitter-rescue J5
+L Transmitter-rescue:Conn_01x02_Male-Connector-Transmitter-rescue-Transmitter-rescue-Transmitter-rescue J5
 U 1 1 60C2BF9E
 P 6800 4900
@@
 $EndComp
 $Comp
-L Transmitter-rescue:+5V-power-Transmitter-rescue-Transmitter-rescue #PWR01
+L Transmitter-rescue:+5V-power-Transmitter-rescue-Transmitter-rescue-Transmitter-rescue #PWR01
 U 1 1 60C2C475
 P 6950 5450
@@
 $EndComp
 $Comp
-L Transmitter-rescue:GND-power-Transmitter-rescue-Transmitter-rescue #PWR02
+L Transmitter-rescue:GND-power-Transmitter-rescue-Transmitter-rescue-Transmitter-rescue #PWR02
 U 1 1 60C2CC2C
 P 7100 5100
@@
 	7000 5000 7100 5000
 $Comp
-L Transmitter-rescue:Conn_01x02_Male-Connector-Transmitter-rescue-Transmitter-rescue J6
+L Transmitter-rescue:Conn_01x02_Male-Connector-Transmitter-rescue-Transmitter-rescue-Transmitter-rescue J6
 U 1 1 60B16252
 P 6050 4900
@@
 $EndComp
 $Comp
-L Transmitter-rescue:SW_SPDT-Switch-Transmitter-rescue-Transmitter-rescue SW1
+L Transmitter-rescue:SW_SPDT-Switch-Transmitter-rescue-Transmitter-rescue-Transmitter-rescue SW1
 U 1 1 60B2577F
 P 6650 5700
